File: PDH.kicad_sch (KiCad schematic)
At the start: 5 parts

Commit message: Jonathan's PDH, swerve, and top-level graphics
Parts:
- removed BT1: 12V, symbol Device:Battery
- removed CB5: CircuitBreaker_1P_US, symbol Device:CircuitBreaker_1P_US
- added F? (x17): 40A, symbol Device:Fuse
- added F? (x4): 10A, symbol Device:Fuse_Small
Other:
- note added: "CAN ID:63"
- note removed: "CIRCUIT 13+"
- moved on the sheet: F1, F2, F3
